File: SampleHolder_Cryo/SampleHolder_Cryo.kicad_pcb (KiCad board)
At the start: 2 copper layers, 30 x 20 mm, 0 parts

Commit message: hola
Parts:
- added P1: GCPW_250, Battery:GCPW_0.254_SH, F.Cu at (155.3, 95.0)
- added P10: GCPW_250, Battery:GCPW_0.254_SH, F.Cu at (135.3, 87.0)
- added P2: GCPW_250, Battery:GCPW_0.254_SH, F.Cu at (164.7, 97.0)
- added P3: GCPW_250, Battery:GCPW_0.254_SH, F.Cu at (144.7, 95.0)
- added P4: GCPW_250, Battery:GCPW_0.254_SH, F.Cu at (135.3, 97.0)
- added P5: DC_Pad, Battery:Pin_Strip, F.Cu at (150.0, 98.8)
- added P6: DC_Pad, Battery:DC_Lines_SH, F.Cu at (150.0, 97.3)
- added P7: GCPW_250, Battery:GCPW_0.254_SH, F.Cu at (155.3, 89.0)
- added P8: GCPW_250, Battery:GCPW_0.254_SH, F.Cu at (164.7, 87.0)
- added P9: GCPW_250, Battery:GCPW_0.254_SH, F.Cu at (144.7, 89.0)
Routing:
- net (no net): track 56.9 -> 0.00 mm
- net Net-(P10-Pad1): track 0.00 -> 9.86 mm
- net Net-(P1-Pad1): track 0.00 -> 9.86 mm
- net Net-(P3-Pad1): track 0.00 -> 9.73 mm
- net Net-(P7-Pad1): track 0.00 -> 9.73 mm
- net Net-(P5-Pad1): track 0.00 -> 3.65 mm
- net Net-(P5-Pad4): track 0.00 -> 3.63 mm
- net Net-(P5-Pad2): track 0.00 -> 2.26 mm
- net Net-(P5-Pad3): track 0.00 -> 2.26 mm
- net GND: vias 0 -> 80
- added copper zone on B.Cu, net GND
- added copper zone on F.Cu, net GND
- removed copper zone on B.Cu, net (none)
- removed copper zone on F.Cu, net (none)
Other:
- board size 30 x 20 mm -> 30 x 15 mm
- net class DC added: clearance 0.125, trace_width 0.2, via_dia 0.8, via_drill 0.4
- net class Default: clearance 0.2 -> 0.196; trace_width 0.25 -> 0.254
- rule trace_clearance: 0.2 -> 0.196
