File: SampleHolder_Cryo/SampleHolder_Cryo.sch (KiCad schematic (older format))
At the start: 0 parts

Commit message: hola
Parts:
- added P1, P10, P2, P3, P4, P7, P8, P9: GCPW_250, Battery:GCPW_0.254_SH, symbol uwRF:GCPW_250
- added P5: DC_Pad, Battery:Pin_Strip, symbol uwRF:DC_Pad
- added P6: DC_Pad, Battery:DC_Lines_SH, symbol uwRF:DC_Pad
Connections:
- net GND: now also P1.2, P1.3, P10.2, P10.3, P2.2, P2.3, P3.2, P3.3, P4.2, P4.3, P7.2, P7.3, P8.2, P8.3, P9.2, P9.3
- new net: P1.1, P2.1
- new net: P3.1, P4.1
- new net: P7.1, P8.1
- new net: P10.1, P9.1
- new net: P5.1, P6.1
- new net: P5.2, P6.2
- new net: P5.3, P6.3
- new net: P5.4, P6.4
